File: additive_vco/additive_vco_hagiwo.brd (EAGLE design)
At the start: 28.1 x 107.5 mm, 41 parts, among them IC1 MCP6232, J1 THONKICONNNEW, J2 THONKICONNNEW, J3 THONKICONNNEW, J4 THONKICONNNEW, M1 ARDUINO-NANO-3.0

Commit message: submit to pcb fab
Parts:
- added C10: 100n, rcl:C025-025X050
- moved D1 1.00 mm to (16.0, 17.5)
- moved D2 1.00 mm to (18.5, 17.5)
- moved D3 1.00 mm to (12.0, 17.5)
- moved D4 1.00 mm to (9.50, 17.5)
Connections:
- new net N$12: IC1.6, IC1.7
- net +5V: now also C10.1
- net GND: now also C10.2, IC1.5
Routing:
- net N$12: track 0.00 -> 2.54 mm
- net A7: track 67.5 -> 68.9 mm
- net N$6: track 25.6 -> 26.1 mm
Other:
- board text added: "github.com/todbot/ eurorack_hagiwo_stuff"
